File: xiao_corne/xiao_corne.kicad_pcb (KiCad board)
At the start: 2 copper layers, 139.5 x 89 mm, 70 parts, among them SW1 SW_Push, SW10 SW_Push, SW11 SW_Push, SW12 SW_Push, SW13 SW_Push, SW17 SW_Push, SW18 SW_Push, SW19 SW_Push, SW2 SW_Push, SW20 SW_Push, SW21 SW_Push, SW22 SW_Push, SW23 SW_Push, SW24 SW_Push, SW25 SW_Push, SW26 SW_Push, SW27 SW_Push, SW3 SW_Push, SW4 SW_Push, SW5 SW_Push, SW9 SW_Push, U1 XIAO-ESP32-S3-SMD, U2 SN74AHCT125DR, U3 MCP1253-33X50I/MS

Commit message: Hardware V0.2
Parts:
- added BT2: Battery, ScottoKeebs_Scotto:Battery, B.Cu at (221.0, 108.0)
- added C4: 10uF, footprints_grm:G-21_MUR, B.Cu at (224.0, 82.8)
- added C5: 10uF, footprints_grm:G-21_MUR, B.Cu at (221.2, 82.8)
- added C6: 1uF, footprints_cl1:CAP_CL10_SAM, B.Cu at (216.4, 83.1)
- added D43: D, ScottoKeebs_Components:Diode_SOD-123, B.Cu at (327.7, 96.8)
- added D44: D, ScottoKeebs_Components:Diode_SOD-123, B.Cu at (269.8, 50.1)
- added D45: D, ScottoKeebs_Components:Diode_SOD-123, B.Cu at (289.1, 91.7)
- added D46: D, ScottoKeebs_Components:Diode_SOD-123, B.Cu at (269.7, 69.7)
- added D47: D, ScottoKeebs_Components:Diode_SOD-123, B.Cu at (215.6, 121.4)
- added D48: D, ScottoKeebs_Components:Diode_SOD-123, B.Cu at (327.7, 77.3)
- added D49: D, ScottoKeebs_Components:Diode_SOD-123, B.Cu at (250.5, 52.6)
- added D50: D, ScottoKeebs_Components:Diode_SOD-123, B.Cu at (259.8, 112.8)
- added D51: D, ScottoKeebs_Components:Diode_SOD-123, B.Cu at (231.1, 74.7)
- added D52: D, ScottoKeebs_Components:Diode_SOD-123, B.Cu at (308.4, 57.5)
- added D53: D, ScottoKeebs_Components:Diode_SOD-123, B.Cu at (231.1, 55.2)
- added D54: D, ScottoKeebs_Components:Diode_SOD-123, B.Cu at (269.7, 89.2)
- added D55: D, ScottoKeebs_Components:Diode_SOD-123, B.Cu at (231.1, 94.3)
- added D56: D, ScottoKeebs_Components:Diode_SOD-123, B.Cu at (308.4, 77.3)
- added D57: D, ScottoKeebs_Components:Diode_SOD-123, B.Cu at (289.1, 52.4)
- added D58: D, ScottoKeebs_Components:Diode_SOD-123, B.Cu at (238.0, 116.6)
- added D59: D, ScottoKeebs_Components:Diode_SOD-123, B.Cu at (250.4, 72.2)
- added D60: D, ScottoKeebs_Components:Diode_SOD-123, B.Cu at (327.7, 57.5)
- added D61: D, ScottoKeebs_Components:Diode_SOD-123, B.Cu at (289.1, 72.2)
- added D62: D, ScottoKeebs_Components:Diode_SOD-123, B.Cu at (308.4, 96.8)
- added D63: D, ScottoKeebs_Components:Diode_SOD-123, B.Cu at (250.4, 91.8)
- added D64: LED_SK6812MINI, ScottoKeebs_Components:LED_SK6812MINI, B.Cu at (238.1, 64.2)
- added D65: LED_SK6812MINI, ScottoKeebs_Components:LED_SK6812MINI, B.Cu at (315.4, 105.8)
- added D66: LED_SK6812MINI, ScottoKeebs_Components:LED_SK6812MINI, B.Cu at (238.1, 103.3)
- added D67: LED_SK6812MINI, ScottoKeebs_Components:LED_SK6812MINI, B.Cu at (257.5, 61.6)
- added D68: LED_SK6812MINI, ScottoKeebs_Components:LED_SK6812MINI, B.Cu at (315.4, 86.3)
- added D69: LED_SK6812MINI, ScottoKeebs_Components:LED_SK6812MINI, B.Cu at (257.4, 100.8)
- added D70: LED_SK6812MINI, ScottoKeebs_Components:LED_SK6812MINI, B.Cu at (276.8, 59.1)
- added D71: LED_SK6812MINI, ScottoKeebs_Components:LED_SK6812MINI, B.Cu at (296.1, 81.2)
- added D72: LED_SK6812MINI, ScottoKeebs_Components:LED_SK6812MINI, B.Cu at (266.8, 121.8)
- added D73: LED_SK6812MINI, ScottoKeebs_Components:LED_SK6812MINI, B.Cu at (296.1, 61.4)
- added D74: LED_SK6812MINI, ScottoKeebs_Components:LED_SK6812MINI, B.Cu at (296.1, 100.7)
- added D75: LED_SK6812MINI, ScottoKeebs_Components:LED_SK6812MINI, B.Cu at (246.9, 124.0)
- added D76: LED_SK6812MINI, ScottoKeebs_Components:LED_SK6812MINI, B.Cu at (315.4, 66.5)
- added D77: LED_SK6812MINI, ScottoKeebs_Components:LED_SK6812MINI, B.Cu at (276.7, 98.2)
- added D78: LED_SK6812MINI, ScottoKeebs_Components:LED_SK6812MINI, B.Cu at (225.6, 126.7)
- added D79: LED_SK6812MINI, ScottoKeebs_Components:LED_SK6812MINI, B.Cu at (334.7, 66.5)
- added D80: LED_SK6812MINI, ScottoKeebs_Components:LED_SK6812MINI, B.Cu at (276.7, 78.7)
- added D81: LED_SK6812MINI, ScottoKeebs_Components:LED_SK6812MINI, B.Cu at (334.7, 86.3)
- added D82: LED_SK6812MINI, ScottoKeebs_Components:LED_SK6812MINI, B.Cu at (257.4, 81.2)
- added D83: LED_SK6812MINI, ScottoKeebs_Components:LED_SK6812MINI, B.Cu at (334.7, 105.8)
- added D84: LED_SK6812MINI, ScottoKeebs_Components:LED_SK6812MINI, B.Cu at (238.1, 83.7)
- added G***: LOGO, LOGO, F.Cu at (188.2, 98.3)
- added G***: LOGO, LOGO, F.Cu at (221.0, 97.9)
- added J1: Conn_01x04_Socket, Connector_PinHeader_2.54mm:PinHeader_1x04_P2.54mm_Vertical, F.Cu at (200.7, 78.2)
- added J2: Conn_01x04_Socket, Connector_PinHeader_2.54mm:PinHeader_1x04_P2.54mm_Vertical, F.Cu at (208.5, 78.2)
- added SW14: SW_Push, ScottoKeebs_Hotswap:Hotswap_Choc_V1V2_1.00u, F.Cu at (276.8, 54.1)
- added SW15: SW_Push, ScottoKeebs_Hotswap:Hotswap_Choc_V1V2_1.00u, F.Cu at (257.5, 56.6)
- added SW16: SW_Push, ScottoKeebs_Hotswap:Hotswap_Choc_V1V2_1.00u, F.Cu at (238.1, 59.2)
- added SW28: SW_Push, ScottoKeebs_Hotswap:Hotswap_Choc_V1V2_1.00u, F.Cu at (296.1, 95.7)
- added SW29: SW_Push, ScottoKeebs_Hotswap:Hotswap_Choc_V1V2_1.00u, F.Cu at (276.7, 73.7)
- added SW30: SW_Push, ScottoKeebs_Hotswap:Hotswap_Choc_V1V2_1.00u, F.Cu at (223.3, 122.1)
- added SW31: SW_Push, ScottoKeebs_Hotswap:Hotswap_Choc_V1V2_1.00u, F.Cu at (266.8, 116.8)
- added SW32: SW_Push, ScottoKeebs_Hotswap:Hotswap_Choc_V1V2_1.00u, F.Cu at (238.1, 78.7)
- added SW33: SW_Push, ScottoKeebs_Hotswap:Hotswap_Choc_V1V2_1.00u, F.Cu at (276.7, 93.2)
- added SW34: SW_Push, ScottoKeebs_Hotswap:Hotswap_Choc_V1V2_1.00u, F.Cu at (238.1, 98.3)
- added SW35: SW_Push, ScottoKeebs_Hotswap:Hotswap_Choc_V1V2_1.00u, F.Cu at (315.4, 81.3)
- added SW36: SW_Push, ScottoKeebs_Hotswap:Hotswap_Choc_V1V2_1.00u, F.Cu at (296.1, 56.4)
- added SW37: SW_Push, ScottoKeebs_Hotswap:Hotswap_Choc_V1V2_1.00u, F.Cu at (245.6, 119.0)
- added SW38: SW_Push, ScottoKeebs_Hotswap:Hotswap_Choc_V1V2_1.00u, F.Cu at (257.4, 76.2)
- added SW39: SW_Push, ScottoKeebs_Hotswap:Hotswap_Choc_V1V2_1.00u, F.Cu at (334.7, 61.5)
- added SW40: SW_Push, ScottoKeebs_Hotswap:Hotswap_Choc_V1V2_1.00u, F.Cu at (296.1, 76.2)
- added SW41: SW_Push, ScottoKeebs_Hotswap:Hotswap_Choc_V1V2_1.00u, F.Cu at (315.4, 100.8)
- added SW42: SW_Push, ScottoKeebs_Hotswap:Hotswap_Choc_V1V2_1.00u, F.Cu at (257.4, 95.8)
- added SW6: SW_Push, ScottoKeebs_Hotswap:Hotswap_Choc_V1V2_1.00u, F.Cu at (334.7, 100.8)
- added SW7: SW_Push, ScottoKeebs_Hotswap:Hotswap_Choc_V1V2_1.00u, F.Cu at (334.7, 81.3)
- added SW8: SW_Push, ScottoKeebs_Hotswap:Hotswap_Choc_V1V2_1.00u, F.Cu at (315.4, 61.5)
- added U4: XIAO-ESP32-S3-SMD, Seeed_Studio_XIAO_Series:XIAO-ESP32-S3-SMD, B.Cu at (226.0, 71.6)
- added U5: MCP1253-33X50I/MS, footprints_mcp:MSOP8_MC_MCH, B.Cu at (218.9, 89.2)
- added U6: SN74AHCT125DR, footprints_sn7:D14, B.Cu at (221.0, 99.3)
- BT1, C1, C2, C3, U1, U2, U3: moved to B.Cu
- moved BT1 34.1 mm to (186.7, 108.0)
- moved U1 16.9 mm to (201.1, 71.6), turned to 180 degrees
- moved U2 11.8 mm to (189.2, 100.6), turned to 180 degrees
- moved U3 11.3 mm to (189.5, 89.9), turned to 90 degrees
- moved C1 10.4 mm to (187.7, 85.1)
- moved C2 9.58 mm to (191.8, 83.6), turned to 180 degrees
- moved C3 3.31 mm to (191.5, 85.6)
Connections:
- net +5V renamed +5V L
- net C1 renamed C1 L
- net C2 renamed C2 L
- net C3 renamed C3 L
- net C4 renamed C4 L
- net C5 renamed C5 L
- net GND renamed GND L
- net LED_3v renamed LED_3v L
- net LED_5v renamed LED_5v L
- net R1 renamed R1 L
- net R2 renamed R2 L
- net R3 renamed R3 L
- net R4 renamed R4 L
- net R5 renamed R5 L
- U1 pad 14: unconnected-(U1-5V-Pad14) -> +5V L USB
Routing:
- net C1: track 0.00 -> 212.9 mm, vias 0 -> 12
- net C5: track 0.00 -> 200.2 mm, vias 0 -> 9
- net C4: track 0.00 -> 194.9 mm, vias 0 -> 7
- net R1: track 0.00 -> 189.9 mm
- net C2: track 0.00 -> 187.7 mm, vias 0 -> 10
- net R3: track 0.00 -> 171.1 mm, vias 0 -> 4
- net C3: track 0.00 -> 165.5 mm, vias 0 -> 9
- net R4: track 0.00 -> 111.3 mm, vias 0 -> 2
- net R2: track 0.00 -> 110.1 mm
- net R5: track 0.00 -> 62.3 mm, vias 0 -> 6
- net GND: track 0.00 -> 57.0 mm, vias 0 -> 28
- net Net-(BT2-+): track 0.00 -> 53.5 mm, vias 0 -> 2
- net LED_3v: track 0.00 -> 44.2 mm
- net Net-(BT1-+): track 13.5 -> 53.0 mm, vias 0 -> 1
- net LED_5v: track 0.00 -> 39.3 mm, vias 0 -> 2
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- added copper zone on B.Cu, net +5V
- added copper zone on F.Cu, net GND
Other:
- board size 139.5 x 89 mm -> 281.7 x 89.1 mm
- board text added: "Zboard V 0.2"

Commit message: Major work for update to 0.3!
Parts:
- removed BT2: Battery, ScottoKeebs_Scotto:Battery
- removed U5: MCP1253-33X50I/MS, footprints_mcp:MSOP8_MC_MCH
- added BT3: Battery, ScottoKeebs_Scotto:Battery, B.Cu at (92.3, 49.1)
- added C10: 10uF, Capacitor_SMD:C_0805_2012Metric, B.Cu at (195.7, 81.2)
- added C7: 1uF, Capacitor_SMD:C_0603_1608Metric, B.Cu at (183.6, 86.0)
- added C8: 10uF, Capacitor_SMD:C_0805_2012Metric, B.Cu at (189.4, 88.8)
- added C9: 10uF, Capacitor_SMD:C_0805_2012Metric, B.Cu at (195.7, 86.6)
- added D85: LED_SK6812MINI, ScottoKeebs_Components:LED_SK6812MINI, B.Cu at (183.0, 107.6)
- added D86: LED_SK6812MINI, ScottoKeebs_Components:LED_SK6812MINI, B.Cu at (187.3, 107.6)
- added D87: LED_SK6812MINI, ScottoKeebs_Components:LED_SK6812MINI, B.Cu at (191.6, 107.6)
- added D88: LED_SK6812MINI, ScottoKeebs_Components:LED_SK6812MINI, B.Cu at (226.2, 107.6)
- added D89: LED_SK6812MINI, ScottoKeebs_Components:LED_SK6812MINI, B.Cu at (221.9, 107.6)
- added D90: LED_SK6812MINI, ScottoKeebs_Components:LED_SK6812MINI, B.Cu at (217.6, 107.6)
- added J10: Conn_01x04_Socket, Connector_PinHeader_2.54mm:PinHeader_1x04_P2.54mm_Vertical, B.Cu at (329.9, 50.9)
- added J3: Conn_01x04_Socket, Connector_PinHeader_2.54mm:PinHeader_1x04_P2.54mm_Vertical, B.Cu at (86.0, 50.8)
- added J4: Conn_01x04_Socket, Connector_PinHeader_2.54mm:PinHeader_1x04_P2.54mm_Vertical, B.Cu at (86.0, 47.2)
- added J5: Conn_01x04_Socket, Connector_PinHeader_2.54mm:PinHeader_1x04_P2.54mm_Vertical, B.Cu at (74.2, 47.2)
- added J6: Conn_01x04_Socket, Connector_PinHeader_2.54mm:PinHeader_1x04_P2.54mm_Vertical, B.Cu at (74.2, 50.8)
- added J7: Conn_01x04_Socket, Connector_PinHeader_2.54mm:PinHeader_1x04_P2.54mm_Vertical, B.Cu at (341.8, 47.4)
- added J8: Conn_01x04_Socket, Connector_PinHeader_2.54mm:PinHeader_1x04_P2.54mm_Vertical, B.Cu at (341.8, 50.9)
- added J9: Conn_01x04_Socket, Connector_PinHeader_2.54mm:PinHeader_1x04_P2.54mm_Vertical, B.Cu at (329.9, 47.4)
- added L1: 2.2uH, Inductor_SMD:L_0805_2012Metric, B.Cu at (183.5, 82.0)
- added L2: 2.2uH, Inductor_SMD:L_0805_2012Metric, B.Cu at (218.9, 81.0)
- added R1: 100k, Resistor_SMD:R_0805_2012Metric, B.Cu at (186.3, 74.4)
- added R2: 100k, Resistor_SMD:R_0805_2012Metric, B.Cu at (195.3, 74.7)
- added R3: 100k, Resistor_SMD:R_0805_2012Metric, B.Cu at (220.3, 74.7)
- added R4: 100k, Resistor_SMD:R_0805_2012Metric, B.Cu at (212.9, 74.8)
- added S1: SLW-864574-5A-RA-N-D, KiCad:SLW8645745ARAND, F.Cu at (119.7, 110.9)
- added S2: SLW-864574-5A-RA-N-D, KiCad:SLW8645745ARAND, F.Cu at (286.8, 113.6)
- added U7: XIAO-HALF-HOLE-23P, xiao ESP32S3 Plus_PCB:MOUDLE23P-SMD-2.54-21X17.8MM.kicad_mod.kicad_sym, B.Cu at (192.7, 58.9)
- C1: value 1uF -> 10uF; footprint footprints_cl1:CAP_CL10_SAM -> Capacitor_SMD:C_0805_2012Metric
- C2, C3: footprint footprints_grm:G-21_MUR -> Capacitor_SMD:C_0805_2012Metric
- C4: value 10uF -> 1uF; footprint footprints_grm:G-21_MUR -> Capacitor_SMD:C_0603_1608Metric
- C5: value 10uF -> 100nF; footprint footprints_grm:G-21_MUR -> Capacitor_SMD:C_0805_2012Metric
- C6: value 1uF -> 100nF; footprint footprints_cl1:CAP_CL10_SAM -> Capacitor_SMD:C_0805_2012Metric
- U1, U4: value XIAO-ESP32-S3-SMD -> TPS61202DRCR; footprint Seeed_Studio_XIAO_Series:XIAO-ESP32-S3-SMD -> TPS61202DRCR:VREG_V62_16624-01YE
- U3: value MCP1253-33X50I/MS -> XIAO-HALF-HOLE-23P; footprint footprints_mcp:MSOP8_MC_MCH -> xiao ESP32S3 Plus_PCB:MOUDLE23P-SMD-2.54-21X17.8MM.kicad_mod.kicad_sym
- moved BT1 142.3 mm to (316.4, 49.3)
- moved U3 41.3 mm to (216.7, 58.9)
- moved C2 32.8 mm to (224.3, 88.2), turned to -90 degrees
- moved C5 31.2 mm to (190.9, 75.6)
- moved C3 28.3 mm to (219.3, 90.6)
- moved C1 25.9 mm to (213.6, 85.4)
- moved U1 16.6 mm to (189.5, 83.4), turned to 0 degrees
- moved U4 15.4 mm to (219.1, 85.4), turned to 0 degrees
- moved C6 7.24 mm to (216.5, 75.8), turned to 90 degrees
- moved U2 3.05 mm to (189.1, 97.5)
- moved C4 1.97 mm to (224.3, 84.8)
- moved U6 1.90 mm to (221.0, 97.4)
Connections:
- BT1 pad 2: GND L -> GND
- C1 pad 1: Net-(U3-C+) -> GND
- C1 pad 2: Net-(U3-C-) -> +5V
- C2 pad 1: Net-(U1-3V3) -> GND
- C2 pad 2: GND L -> +5V
- C3 pad 1: +5V L -> GND
- C3 pad 2: GND L -> +3.3V
- C4 pad 1: +5V -> GND
- C4 pad 2: GND -> +3.3V
- C5 pad 1: Net-(U4-3V3) -> GND L
- C5 pad 2: GND -> Net-(C5-Pad2)
- C6 pad 1: Net-(U5-C+) -> GND
- D42 pad 2: unconnected-(D42-DOUT-Pad2) -> Net-(D42-DOUT)
- D78 pad 2: unconnected-(D78-DOUT-Pad2) -> Net-(D78-DOUT)
- U1 pad 1: R1 L -> Net-(U1-VAUX)
- U1 pad 10: C5 L -> +5V L
- U1 pad 11: LED_3v L -> unconnected-(U1-EP-Pad11)
- U1 pad 12: Net-(U1-3V3) -> (no net)
- U1 pad 13: GND L -> (no net)
- U1 pad 14: +5V L USB -> (no net)
- U1 pad 15: Net-(BT1-+) -> (no net)
- U1 pad 2: R2 L -> +5V L
- U1 pad 3: R3 L -> Net-(U1-L)
- U1 pad 4: R4 L -> GND L
- U1 pad 5: R5 L -> +3.3V L
- U1 pad 6: C1 L -> +3.3V L
- U1 pad 7: C2 L -> +3.3V L
- U1 pad 8: C3 L -> +3.3V L
- U1 pad 9: C4 L -> GND L
- U3 pad 1: unconnected-(U3-PGOOD-Pad1) -> R1
- U3 pad 2: +5V L -> R2
- U3 pad 3: Net-(U1-3V3) -> R3
- U3 pad 4: GND L -> R4
- U3 pad 5: Net-(U3-C-) -> R5
- U3 pad 6: Net-(U3-C+) -> C1
- U3 pad 7: Net-(U1-3V3) -> C2
- U3 pad 8: GND L -> C3
- U4 pad 1: R1 -> +3.3V
- U4 pad 10: C5 -> +5V
- U4 pad 11: LED_3v -> unconnected-(U4-EP-Pad11)
- U4 pad 12: Net-(U4-3V3) -> (no net)
- U4 pad 13: GND -> (no net)
- U4 pad 14: +5V USB -> (no net)
- U4 pad 15: Net-(BT2-+) -> (no net)
- U4 pad 2: R2 -> +5V
- U4 pad 3: R3 -> Net-(U4-L)
- U4 pad 4: R4 -> GND
- U4 pad 5: R5 -> +3.3V
- U4 pad 6: C1 -> +3.3V
- U4 pad 7: C2 -> +3.3V
- U4 pad 8: C3 -> +3.3V
- U4 pad 9: C4 -> GND
Routing:
- net +3.3V: track 0.00 -> 206.9 mm, vias 0 -> 9
- net GND L: track 91.7 -> 280.8 mm, vias 27 -> 45
- net +3.3V L: track 0.00 -> 179.8 mm, vias 0 -> 6
- net GPIO_4_L: track 0.00 -> 166.6 mm, vias 0 -> 1
- net GPIO_1: track 0.00 -> 162.2 mm, vias 0 -> 1
- net GPIO_3_L: track 0.00 -> 161.8 mm, vias 0 -> 3
- net GPIO_1_L: track 0.00 -> 160.7 mm, vias 0 -> 4
- net GPIO_6: track 0.00 -> 160.5 mm, vias 0 -> 1
- net GPIO_2_L: track 0.00 -> 158.8 mm, vias 0 -> 3
- net GPIO_7: track 0.00 -> 151.5 mm, vias 0 -> 1
- net Net-(U7-BAT+): track 0.00 -> 150.5 mm, vias 0 -> 2
- net GPIO_8: track 0.00 -> 150.2 mm, vias 0 -> 1
- net GPIO_2: track 0.00 -> 145.9 mm, vias 0 -> 2
- net GPIO_5_L: track 0.00 -> 144.6 mm, vias 0 -> 1
- net GPIO_8_L: track 0.00 -> 143.3 mm, vias 0 -> 4
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Other:
- outline, holes or cut-outs redrawn
- board text added: "Zboard V 0.3"
- board text removed: "Zboard V 0.2"
