File: xiao_corne/xiao_corne.kicad_pcb (KiCad board)
At the start: 2 copper layers, 281.7 x 89.1 mm, 170 parts, among them J1 Conn_01x04_Socket, J10 Conn_01x04_Socket, J2 Conn_01x04_Socket, J3 Conn_01x04_Socket, J4 Conn_01x04_Socket, J5 Conn_01x04_Socket, J6 Conn_01x04_Socket, J7 Conn_01x04_Socket, J8 Conn_01x04_Socket, J9 Conn_01x04_Socket, SW1 SW_Push, SW10 SW_Push, SW11 SW_Push, SW12 SW_Push, SW13 SW_Push, SW14 SW_Push, SW15 SW_Push, SW16 SW_Push, SW17 SW_Push, SW18 SW_Push, SW19 SW_Push, SW2 SW_Push, SW20 SW_Push, SW21 SW_Push, SW22 SW_Push, SW23 SW_Push, SW24 SW_Push, SW25 SW_Push, SW26 SW_Push, SW27 SW_Push, SW28 SW_Push, SW29 SW_Push, SW3 SW_Push, SW30 SW_Push, SW31 SW_Push, SW32 SW_Push, SW33 SW_Push, SW34 SW_Push, SW35 SW_Push, SW36 SW_Push, SW37 SW_Push, SW38 SW_Push, SW39 SW_Push, SW4 SW_Push, SW40 SW_Push, SW41 SW_Push, SW42 SW_Push, SW5 SW_Push, SW6 SW_Push, SW7 SW_Push, SW8 SW_Push, SW9 SW_Push, U1 TPS61202DRCR, U2 SN74AHCT125DR, U3 XIAO-HALF-HOLE-23P, U4 TPS61202DRCR, U6 SN74AHCT125DR, U7 XIAO-HALF-HOLE-23P

Commit message: Fixed issue with battery voltage monitor
Parts:
- renumbered BT3 to BT1, BT1 to BT2, C8 to C1, C6 to C10, C9 to C2, C1 to C3, C2 to C4, C10 to C5, C7 to C6, C3 to C7, C4 to C8, C5 to C9, D60 to D10, D9 to D11, D10 to D12, D11 to D13, D12 to D14, D13 to D15, D6 to D16, D7 to D17, D8 to D18, D14 to D19, D15 to D20, D16 to D21, D28 to D22, D29 to D23, D44 to D24, D49 to D25, D53 to D26, D57 to D27, D61 to D28, D64 to D29, D67 to D30, D70 to D31, D73 to D32, D76 to D33, D79 to D34, D81 to D35, D83 to D36, D17 to D37, D18 to D38, D19 to D39, D20 to D40, D21 to D41, D45 to D42, D50 to D43, D54 to D44, D58 to D45, D62 to D46, D30 to D47, D31 to D48, D32 to D49, D33 to D50, D34 to D51, D35 to D52, D36 to D53, D37 to D54, D65 to D55, D68 to D56, D71 to D57, D74 to D58, D77 to D59, D43 to D6, D80 to D60, D82 to D61, D84 to D62, D22 to D63, D23 to D64, D24 to D65, D25 to D66, D26 to D67, D46 to D68, D51 to D69, D48 to D7, D55 to D70, D59 to D71, D63 to D72, D38 to D73, D39 to D74, D40 to D75, D41 to D76, D42 to D77, D85 to D78, D86 to D79, D52 to D8, D87 to D80, D66 to D81, D69 to D82, D72 to D83, D75 to D84, D78 to D85, D88 to D86, D89 to D87, D90 to D88, D27 to D89, D56 to D9, D47 to D90, J2 to J1, J6 to J10, J7 to J2, J8 to J3, J3 to J5, J1 to J6, J9 to J7, J10 to J8, J5 to J9, R3 to R2, R2 to R3, SW39 to SW10, SW9 to SW11, SW10 to SW12, SW11 to SW13, SW12 to SW14, SW13 to SW15, SW14 to SW16, SW15 to SW17, SW16 to SW18, SW36 to SW19, SW40 to SW20, SW17 to SW21, SW18 to SW22, SW19 to SW23, SW20 to SW24, SW21 to SW25, SW28 to SW26, SW31 to SW27, SW33 to SW28, SW37 to SW29, SW41 to SW30, SW22 to SW31, SW23 to SW32, SW24 to SW33, SW25 to SW34, SW26 to SW35, SW29 to SW36, SW32 to SW37, SW34 to SW38, SW38 to SW39, SW42 to SW40, SW27 to SW41, SW30 to SW42, SW35 to SW9, U2 to U1, U6 to U2, U7 to U3, U3 to U4, U1 to U5, U4 to U6
Connections:
- C10 pad 2: Net-(C6-Pad2) -> Net-(U4-GPIO10_XMCLK/ADC_BAT)
- C9 pad 2: Net-(C5-Pad2) -> Net-(U3-GPIO10_XMCLK/ADC_BAT)
- R1 pad 1: Net-(C5-Pad2) -> Net-(U3-GPIO10_XMCLK/ADC_BAT)
- R1 pad 2: Net-(U7-GPIO10_XMCLK/ADC_BAT) -> GND L
- R2 pad 1: Net-(C6-Pad2) -> Net-(U4-GPIO10_XMCLK/ADC_BAT)
- R2 pad 2: Net-(U3-GPIO10_XMCLK/ADC_BAT) -> GND
- R3 pad 1: Net-(C5-Pad2) -> Net-(U3-GPIO10_XMCLK/ADC_BAT)
- R4 pad 1: Net-(C6-Pad2) -> Net-(U4-GPIO10_XMCLK/ADC_BAT)
- U3 pad 20: Net-(U7-GPIO10_XMCLK/ADC_BAT) -> Net-(U3-GPIO10_XMCLK/ADC_BAT)
- U4 pad 20: Net-(U3-GPIO10_XMCLK/ADC_BAT) -> Net-(U4-GPIO10_XMCLK/ADC_BAT)
Routing:
- net Net-(U7-GPIO10_XMCLK/ADC_BAT): track 24.6 -> 0.00 mm
- net Net-(U4-GPIO10_XMCLK/ADC_BAT): track 0.00 -> 16.2 mm, vias 0 -> 2
- net GND: track 84.2 -> 96.8 mm, vias 37 -> 38
- net Net-(U3-GPIO10_XMCLK/ADC_BAT): track 12.9 -> 22.4 mm, vias 2 -> 0
- net Net-(C5-Pad2): track 6.94 -> 0.00 mm
- net GND L: track 280.8 -> 287.1 mm
- net Net-(C6-Pad2): track 5.62 -> 0.00 mm

Commit message: V4
Other:
- board text added: "Zboard V 0.4"
- board text removed: "Zboard V 0.3"
Changed lines of the file:
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@@
 		(layer "Edge.Cuts")
 	)
-	(gr_text "Zboard V 0.3"
+	(gr_text "Zboard V 0.4"
 		(at 202.184 61.214 90)
 		(layer "F.SilkS")
@@
 			(justify bottom)
 		)
-		(render_cache "Zboard V 0.3" 90
+		(render_cache "Zboard V 0.4" 90
 			(polygon
 				(pts
@@
 			(polygon
 				(pts
-					(xy 200.292813 52.847705) (xy 200.395127 52.856165) (xy 200.482647 52.880221) (xy 200.558039 52.918831)
-					(xy 200.623274 52.972269) (xy 200.696082 53.060875) (xy 200.751955 53.16241) (xy 200.791191 53.278916)
-					(xy 200.799617 53.278916) (xy 200.830743 53.12267) (xy 200.880068 53.003399) (xy 200.945186 52.913528)
-					(xy 201.007804 52.859836) (xy 201.080035 52.821233) (xy 201.163765 52.797261) (xy 201.261602 52.788842)
-					(xy 201.374923 52.798597) (xy 201.478352 52.827134) (xy 201.573867 52.874327) (xy 201.657522 52.939414)
-					(xy 201.730216 53.025933) (xy 201.79222 53.137499) (xy 201.834309 53.258748) (xy 201.861913 53.409372)
-					(xy 201.871965 53.595332) (xy 201.85911 53.80963) (xy 201.822159 54.000834) (xy 201.762789 54.172112)
-					(xy 201.404362 54.172112) (xy 201.461067 54.040272) (xy 201.502426 53.901857) (xy 201.528017 53.762512)
-					(xy 201.536009 53.640029) (xy 201.525102 53.489747) (xy 201.497264 53.388294) (xy 201.457607 53.322269)
-					(xy 201.399733 53.27267) (xy 201.327476 53.242166) (xy 201.236445 53.231288) (xy 201.157591 53.242239)
-					(xy 201.095029 53.273298) (xy 201.0471 53.326956) (xy 201.0082 53.420332) (xy 200.987211 53.53563)
-					(xy 200.978769 53.712935) (xy 200.978769 53.864122) (xy 200.654048 53.864122) (xy 200.654048 53.710126)
-					(xy 200.643875 53.536533) (xy 200.619 53.428637) (xy 200.575198 53.344118) (xy 200.523745 53.297112)
-					(xy 200.460023 53.271081) (xy 200.385259 53.262063) (xy 200.317145 53.269934) (xy 200.262619 53.292034)
-					(xy 200.218563 53.327886) (xy 200.187638 53.375799) (xy 200.166497 53.446382) (xy 200.158357 53.547705)
-					(xy 200.171285 53.684283) (xy 200.20745 53.795489) (xy 200.2579 53.895783) (xy 200.304048 53.973298)
-					(xy 200.012789 54.169303) (xy 199.937102 54.044138) (xy 199.872838 53.893553) (xy 199.842809 53.7866)
-					(xy 199.823605 53.661958) (xy 199.816784 53.51693) (xy 199.825737 53.361012) (xy 199.850765 53.230072)
-					(xy 199.889745 53.120265) (xy 199.94147 53.028323) (xy 200.010778 52.948728) (xy 200.090806 52.893262)
-					(xy 200.183632 52.859489)
+					(xy 201.429642 52.965308) (xy 201.844 52.965308) (xy 201.844 53.376857) (xy 201.429642 53.376857)
+					(xy 201.429642 54.230852) (xy 201.135573 54.230852) (xy 199.869394 53.37124) (xy 200.329205 53.37124)
+					(xy 200.438504 53.424484) (xy 200.547558 53.491651) (xy 201.10199 53.858504) (xy 201.10199 53.376857)
+					(xy 200.763225 53.376857) (xy 200.606421 53.374048) (xy 200.43423 53.367087) (xy 200.329205 53.360126)
+					(xy 200.329205 53.37124) (xy 199.869394 53.37124) (xy 199.84475 53.354509) (xy 199.84475 52.965308)
+					(xy 201.10199 52.965308) (xy 201.10199 52.724484) (xy 201.429642 52.724484)
 				)
 			)
 		)
 	)
-	(gr_text "Zboard V 0.3"
+	(gr_text "Zboard V 0.4"
 		(at 205.74 61.468 270)
 		(layer "F.SilkS")
@@
 			(justify bottom)
 		)
-		(render_cache "Zboard V 0.3" 270
+		(render_cache "Zboard V 0.4" 270
 			(polygon
 				(pts
@@
 			(polygon
 				(pts
-					(xy 207.631186 69.834294) (xy 207.528872 69.825834) (xy 207.441352 69.801778) (xy 207.36596 69.763168)
-					(xy 207.300725 69.70973) (xy 207.227917 69.621124) (xy 207.172044 69.519589) (xy 207.132808 69.403083)
-					(xy 207.124382 69.403083) (xy 207.093256 69.559329) (xy 207.043931 69.6786) (xy 206.978813 69.768471)
-					(xy 206.916195 69.822163) (xy 206.843964 69.860766) (xy 206.760234 69.884738) (xy 206.662397 69.893157)
-					(xy 206.549076 69.883402) (xy 206.445647 69.854865) (xy 206.350132 69.807672) (xy 206.266477 69.742585)
-					(xy 206.193783 69.656066) (xy 206.131779 69.5445) (xy 206.08969 69.423251) (xy 206.062086 69.272627)
-					(xy 206.052034 69.086667) (xy 206.064889 68.872369) (xy 206.10184 68.681165) (xy 206.16121 68.509887)
-					(xy 206.519637 68.509887) (xy 206.462932 68.641727) (xy 206.421573 68.780142) (xy 206.395982 68.919487)
-					(xy 206.38799 69.04197) (xy 206.398897 69.192252) (xy 206.426735 69.293705) (xy 206.466392 69.35973)
-					(xy 206.524266 69.409329) (xy 206.596523 69.439833) (xy 206.687554 69.450711) (xy 206.766408 69.43976)
-					(xy 206.82897 69.408701) (xy 206.876899 69.355043) (xy 206.915799 69.261667) (xy 206.936788 69.146369)
-					(xy 206.94523 68.969064) (xy 206.94523 68.817877) (xy 207.269951 68.817877) (xy 207.269951 68.971873)
-					(xy 207.280124 69.145466) (xy 207.305 69.253362) (xy 207.348801 69.337881) (xy 207.400254 69.384887)
-					(xy 207.463976 69.410918) (xy 207.53874 69.419936) (xy 207.606854 69.412065) (xy 207.66138 69.389965)
-					(xy 207.705436 69.354113) (xy 207.736361 69.3062) (xy 207.757502 69.235617) (xy 207.765642 69.134294)
-					(xy 207.752714 68.997716) (xy 207.716549 68.88651) (xy 207.666099 68.786216) (xy 207.619951 68.708701)
-					(xy 207.91121 68.512696) (xy 207.986897 68.637861) (xy 208.051161 68.788446) (xy 208.08119 68.895399)
-					(xy 208.100394 69.020041) (xy 208.107215 69.165069) (xy 208.098262 69.320987) (xy 208.073234 69.451927)
-					(xy 208.034254 69.561734) (xy 207.982529 69.653676) (xy 207.913221 69.733271) (xy 207.833193 69.788737)
-					(xy 207.740367 69.82251)
-				)
-			)
+					(xy 208.079249 69.32749) (xy 208.079249 69.716691) (xy 206.822009 69.716691) (xy 206.822009 69.957515)
+					(xy 206.494357 69.957515) (xy 206.494357 69.716691) (xy 206.08 69.716691) (xy 206.08 69.305142)
+					(xy 206.494357 69.305142) (xy 206.822009 69.305142) (xy 207.160774 69.305142) (xy 207.317578 69.307951)
+					(xy 207.489769 69.314912) (xy 207.594794 69.321873) (xy 207.594794 69.310759) (xy 207.485495 69.257515)
+					(xy 207.376441 69.190348) (xy 206.822009 68.823495) (xy 206.822009 69.305142) (xy 206.494357 69.305142)
+					(xy 206.494357 68.451147) (xy 206.788426 68.451147)
+				)
+			)

Commit message: starting layout for left side
Parts:
- removed BT2: Battery, ScottoKeebs_Scotto:Battery
- removed C1, C2, C5: 10uF, Capacitor_SMD:C_0805_2012Metric
- removed C6: 1uF, Capacitor_SMD:C_0603_1608Metric
- removed D10, D11, D12, D13, D14, D15, D24, D25, D26, D27, D28, D3, D37, D38, D39, D4, D40, D41, D42, D43, D44, D45, D46, D5, D6, D63, D64, D65, D66, D67, D68, D69, D7, D70, D71, D72, D8, D89, D9, D90: D, ScottoKeebs_Components:Diode_SOD-123
- removed D29, D30, D31, D32, D33, D34, D35, D36, D55, D56, D57, D58, D59, D60, D61, D62, D78, D79, D80, D81, D82, D83, D84, D85, D86, D87, D88: LED_SK6812MINI, ScottoKeebs_Components:LED_SK6812MINI
- removed the G*** at (188.2, 98.3)
- removed the G*** at (221.0, 97.9)
- removed J10, J2, J3, J4, J5, J7, J8, J9: Conn_01x04_Socket, Connector_PinHeader_2.54mm:PinHeader_1x04_P2.54mm_Vertical
- removed L1: 2.2uH, Inductor_SMD:L_0805_2012Metric
- removed S2: SLW-864574-5A-RA-N-D, KiCad:SLW8645745ARAND
- removed SW10, SW16, SW17, SW18, SW19, SW20, SW26, SW27, SW28, SW29, SW30, SW36, SW37, SW38, SW39, SW40, SW42, SW7, SW8, SW9: SW_Push, ScottoKeebs_Hotswap:Hotswap_Choc_V1V2_1.00u
- removed U5, U6: TPS61202DRCR, TPS61202DRCR:VREG_V62_16624-01YE
- added C11: 0.1uF, Capacitor_SMD:C_0805_2012Metric, F.Cu at (293.1, 152.6)
- added C12: 10uF, Capacitor_SMD:C_0805_2012Metric, F.Cu at (310.7, 146.6)
- added C13: 10uF, Capacitor_SMD:C_0805_2012Metric, F.Cu at (302.7, 140.1)
- added C14: 4.7u, Capacitor_SMD:C_0805_2012Metric, F.Cu at (377.7, 141.6)
- added C15: 4.7u, Capacitor_SMD:C_0805_2012Metric, F.Cu at (371.2, 142.1)
- added C16: 4.7u, Capacitor_SMD:C_0805_2012Metric, F.Cu at (361.7, 134.1)
- added G***: LOGO, LOGO, F.Cu at (254.9, 204.8)
- added G***: LOGO, LOGO, F.Cu at (287.6, 204.4)
- added H1: MountingHole_Pad, MountingHole:MountingHole_3.2mm_M3_ISO14580, F.Cu at (64.0, 81.2)
- added H2: MountingHole_Pad, MountingHole:MountingHole_3.2mm_M3_ISO14580, F.Cu at (155.1, 119.1)
- added H3: MountingHole_Pad, MountingHole:MountingHole_3.2mm_M3_ISO14580, F.Cu at (140.1, 77.6)
- added R10: 10k, Resistor_SMD:R_0805_2012Metric, F.Cu at (380.7, 125.1)
- added R5: 5.1k, Resistor_SMD:R_0805_2012Metric, F.Cu at (212.6, 51.1)
- added R6: 5.1k, Resistor_SMD:R_0805_2012Metric, F.Cu at (207.2, 51.1)
- added R7: 10k, Resistor_SMD:R_0805_2012Metric, F.Cu at (171.0, 79.6)
- added R8: 10k, Resistor_SMD:R_0805_2012Metric, F.Cu at (192.5, 110.1)
- added R9: 10k, Resistor_SMD:R_0805_2012Metric, F.Cu at (384.2, 131.1)
- BT1: footprint ScottoKeebs_Scotto:Battery -> Connector_PinHeader_2.00mm:PinHeader_1x02_P2.00mm_Vertical; moved to F.Cu
- C10: value 100nF -> 10uF; moved to F.Cu
- C3: value 10uF -> 1u; moved to F.Cu
- C4: value 10uF -> 22u; moved to F.Cu
- C7: value 10uF -> 0.1u; moved to F.Cu
- C8: value 1uF -> 100nF; footprint Capacitor_SMD:C_0603_1608Metric -> Capacitor_SMD:C_0805_2012Metric; moved to F.Cu
- C9, L2, R1, R3: moved to F.Cu
- D1, D2: value D -> ESD321DPYR; footprint ScottoKeebs_Components:Diode_SOD-123 -> ESD321DPYR:TVS_ESD321DPYR; moved to F.Cu
- D16, D17, D18, D19, D20, D21, D22, D23, D47, D48, D49, D50, D51, D52, D53, D54, D73, D74, D75, D76, D77: footprint ScottoKeebs_Components:LED_SK6812MINI -> footprints:LED_SK6812MINI; moved to F.Cu
- J1: value Conn_01x04_Socket -> USB4110GFA; footprint Connector_PinHeader_2.54mm:PinHeader_1x04_P2.54mm_Vertical -> USB4110_GF_A:GCT_USB4110GFA
- R2, R4: value 100k -> 22; moved to F.Cu
- S1: footprint KiCad:SLW8645745ARAND -> SLW_864574_5A_RA_N_D:SW_SLW-864574-5A-RA-N-D
- SW1, SW11, SW12, SW13, SW14, SW15, SW2, SW21, SW22, SW23, SW24, SW25, SW3, SW31, SW32, SW33, SW34, SW35, SW4, SW41, SW5: footprint ScottoKeebs_Hotswap:Hotswap_Choc_V1V2_1.00u -> footprints:Hotswap_Choc_V1V2
- SW6: footprint ScottoKeebs_Hotswap:Hotswap_Choc_V1V2_1.00u -> footprints:MJTP1117
- U1: footprint footprints_sn7:D14 -> footprints-sn7:D14; moved to F.Cu
- U2: value SN74AHCT125DR -> ESP32-S3-WROOM-1; footprint footprints_sn7:D14 -> PCM_Espressif:ESP32-S3-WROOM-1; moved to F.Cu
- U3: value XIAO-HALF-HOLE-23P -> TPS61201DRCT; footprint xiao ESP32S3 Plus_PCB:MOUDLE23P-SMD-2.54-21X17.8MM.kicad_mod.kicad_sym -> TPS61201DRCT:VREG_V62_16624-01YE; moved to F.Cu
- U4: value XIAO-HALF-HOLE-23P -> BQ24232RGTR; footprint xiao ESP32S3 Plus_PCB:MOUDLE23P-SMD-2.54-21X17.8MM.kicad_mod.kicad_sym -> BQ24232RGTR:RGT0016C; moved to F.Cu
- moved D23 243.2 mm to (252.0, -59.9), turned to -90 degrees
- moved D22 233.6 mm to (256.1, -59.9), turned to -90 degrees
- moved D47 226.4 mm to (247.9, -59.9), turned to -90 degrees
- moved D21 225.3 mm to (260.3, -59.9), turned to -90 degrees
- moved D20 212.8 mm to (264.4, -59.9), turned to -90 degrees
- moved D48 209.6 mm to (243.7, -59.9), turned to -90 degrees
- moved D50 202.1 mm to (235.5, -59.9), turned to -90 degrees
- moved D19 197.6 mm to (268.5, -59.9), turned to -90 degrees
- moved D75 192.9 mm to (206.6, -60.1), turned to -90 degrees
- moved D49 189.7 mm to (239.6, -59.9), turned to -90 degrees
- moved D76 188.1 mm to (202.5, -60.1), turned to -90 degrees
- moved D77 187.1 mm to (198.4, -60.1), turned to -90 degrees
- moved D51 186.5 mm to (231.4, -59.9), turned to -90 degrees
- moved D18 184.0 mm to (272.6, -59.9), turned to -90 degrees
- moved U1 175.7 mm to (359.2, 53.4), turned to 0 degrees
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Connections:
- C10 pad 1: GND -> GND L
- C10 pad 2: Net-(U4-GPIO10_XMCLK/ADC_BAT) -> +4.4V L
- C3 pad 1: GND -> GND L
- C3 pad 2: +5V -> Net-(U2-EN)
- C4 pad 1: GND -> GND L
- C4 pad 2: +5V -> +3.3V L
- C7 pad 1: GND -> GND L
- C7 pad 2: +3.3V -> +3.3V L
- C8 pad 1: GND -> Net-(U2-GPIO0/BOOT)
- C8 pad 2: +3.3V -> GND L
- C9 pad 2: Net-(U3-GPIO10_XMCLK/ADC_BAT) -> BAT/2 MON L
- D1 pad 1: Net-(D1-K) -> Net-(J1-DN1)
- D1 pad 2: C1 L -> GND L
- D16 pad 1: +5V L -> +4.4V L
- D17 pad 1: +5V L -> +4.4V L
- D18 pad 1: +5V L -> +4.4V L
- D19 pad 1: +5V L -> +4.4V L
- D2 pad 1: Net-(D2-K) -> Net-(J1-DP1)
- D2 pad 2: C2 L -> GND L
- D20 pad 1: +5V L -> +4.4V L
- D21 pad 1: +5V L -> +4.4V L
- D22 pad 1: +5V L -> +4.4V L
- D23 pad 1: +5V L -> +4.4V L
- D47 pad 1: +5V L -> +4.4V L
- D48 pad 1: +5V L -> +4.4V L
- D49 pad 1: +5V L -> +4.4V L
- D50 pad 1: +5V L -> +4.4V L
- D51 pad 1: +5V L -> +4.4V L
- D52 pad 1: +5V L -> +4.4V L
- D53 pad 1: +5V L -> +4.4V L
- D54 pad 1: +5V L -> +4.4V L
- D73 pad 1: +5V L -> +4.4V L
- D74 pad 1: +5V L -> +4.4V L
- D75 pad 1: +5V L -> +4.4V L
- D76 pad 1: +5V L -> +4.4V L
- D77 pad 1: +5V L -> +4.4V L
- D77 pad 2: Net-(D77-DOUT) -> unconnected-(D77-DOUT-Pad2)
- J6 pad 1: +5V L USB -> VUSB L
- L2 pad 1: Net-(U6-L) -> Net-(U3-L)
- L2 pad 2: +3.3V -> +4.4V L
- R1 pad 1: Net-(U3-GPIO10_XMCLK/ADC_BAT) -> GND L
- R1 pad 2: GND L -> BAT/2 MON L
- R2 pad 1: Net-(U4-GPIO10_XMCLK/ADC_BAT) -> Net-(U2-GPIO20/U1CTS/ADC2_CH9/CLK_OUT1/USB_D+)
- R2 pad 2: GND -> Net-(J1-DP1)
- R3 pad 1: Net-(U3-GPIO10_XMCLK/ADC_BAT) -> BAT/2 MON L
- R3 pad 2: Net-(U3-BAT+) -> VBAT L
- R4 pad 1: Net-(U4-GPIO10_XMCLK/ADC_BAT) -> Net-(U2-GPIO19/U1RTS/ADC2_CH8/CLK_OUT2/USB_D-)
- R4 pad 2: Net-(U4-BAT+) -> Net-(J1-DN1)
- S1 pad 2: Net-(U3-BAT+) -> VBAT L
- SW1 pad 1: Net-(D1-K) -> +3.3V L
- SW1 pad 2: R1 L -> KS_L1
- SW11 pad 1: Net-(D11-K) -> +3.3V L
- SW11 pad 2: R2 L -> KS_L6
- SW12 pad 1: Net-(D12-K) -> +3.3V L
- SW12 pad 2: R2 L -> KS_L7
- SW13 pad 1: Net-(D13-K) -> +3.3V L
- SW13 pad 2: R2 L -> KS_L8
- SW14 pad 1: Net-(D14-K) -> +3.3V L
- SW14 pad 2: R2 L -> KS_L9
- SW15 pad 1: Net-(D15-K) -> +3.3V L
- SW15 pad 2: R2 L -> KS_L10
- SW2 pad 1: Net-(D2-K) -> +3.3V L
- SW2 pad 2: R1 L -> KS_L2
- SW21 pad 1: Net-(D37-K) -> +3.3V L
- SW21 pad 2: R3 L -> KS_L11
- SW22 pad 1: Net-(D38-K) -> +3.3V L
- SW22 pad 2: R3 L -> KS_L12
- SW23 pad 1: Net-(D39-K) -> +3.3V L
- SW23 pad 2: R3 L -> KS_L13
- SW24 pad 1: Net-(D40-K) -> +3.3V L
- SW24 pad 2: R3 L -> KS_L14
- SW25 pad 1: Net-(D41-K) -> +3.3V L
- SW25 pad 2: R3 L -> KS_L15
- SW3 pad 1: Net-(D3-K) -> +3.3V L
- SW3 pad 2: R1 L -> KS_L3
- SW31 pad 1: Net-(D63-K) -> +3.3V L
- SW31 pad 2: R4 L -> KS_L16
- SW32 pad 1: Net-(D64-K) -> +3.3V L
- SW32 pad 2: R4 L -> KS_L17
- SW33 pad 1: Net-(D65-K) -> +3.3V L
- SW33 pad 2: R4 L -> KS_L18
- SW34 pad 1: Net-(D66-K) -> +3.3V L
- SW34 pad 2: R4 L -> KS_L19
- SW35 pad 1: Net-(D67-K) -> +3.3V L
- SW35 pad 2: R4 L -> KS_L20
- SW4 pad 1: Net-(D4-K) -> +3.3V L
- SW4 pad 2: R1 L -> KS_L4
- SW41 pad 1: Net-(D89-K) -> +3.3V L
- SW41 pad 2: R5 L -> KS_L21
- SW5 pad 1: Net-(D5-K) -> +3.3V L
- SW5 pad 2: R1 L -> KS_L5
- SW6 pad 1: Net-(D6-K) -> GND L
- SW6 pad 2: R1 -> Net-(U2-GPIO0/BOOT)
- U1 pad 14: +5V L -> +4.4V L
- U2 pad 10: unconnected-(U2-*3OE-Pad10) -> KS_L14
- U2 pad 11: unconnected-(U2-4Y-Pad11) -> KS_L15
- U2 pad 12: unconnected-(U2-4A-Pad12) -> KS_L7
- U2 pad 13: unconnected-(U2-*4OE-Pad13) -> Net-(U2-GPIO19/U1RTS/ADC2_CH8/CLK_OUT2/USB_D-)
- U2 pad 14: +5V -> Net-(U2-GPIO20/U1CTS/ADC2_CH9/CLK_OUT1/USB_D+)
- U2 pad 2: LED_3v -> +3.3V L
- U2 pad 3: LED_5v -> Net-(U2-EN)
- U2 pad 4: unconnected-(U2-*2OE-Pad4) -> KS_L3
- U2 pad 5: unconnected-(U2-2A-Pad5) -> KS_L4
- U2 pad 6: unconnected-(U2-2Y-Pad6) -> KS_L5
- U2 pad 7: GND -> KS_L6
- U3 pad 1: R1 L -> Net-(U3-VAUX)
- U3 pad 10: C5 L -> +3.3V L
- U3 pad 11: LED_3v L -> unconnected-(U3-EP-Pad11)
- U3 pad 12: +3.3V L -> (no net)
- U3 pad 13: GND L -> (no net)
- U3 pad 14: +5V L USB -> (no net)
- U3 pad 15: GPIO_1_L -> (no net)
- U3 pad 2: R2 L -> +3.3V L
- U3 pad 3: R3 L -> Net-(U3-L)
- U3 pad 4: R4 L -> GND L
- U3 pad 5: R5 L -> +4.4V L
- U3 pad 6: C1 L -> +4.4V L
- U3 pad 7: C2 L -> +4.4V L
- U3 pad 8: C3 L -> +4.4V L
- U3 pad 9: C4 L -> GND L
- U4 pad 1: R1 -> Net-(U4-TS)
- U4 pad 10: C5 -> +4.4V L
- U4 pad 11: LED_3v -> +4.4V L
- U4 pad 12: +3.3V -> unconnected-(U4-ILIM-Pad12)
- U4 pad 13: GND -> VUSB L
- U4 pad 14: +5V USB -> unconnected-(U4-TMR-Pad14)
- U4 pad 15: GPIO_1 -> unconnected-(U4-ITERM-Pad15)
- U4 pad 16: GPIO_2 -> Net-(U4-ISET)
- U4 pad 17: GPIO_3 -> GND L
- U4 pad 2: R2 -> VBAT L
- U4 pad 3: R3 -> VBAT L
- U4 pad 4: R4 -> GND
- U4 pad 5: R5 -> GND L
- U4 pad 6: C1 -> +4.4V L
- U4 pad 7: C2 -> pgood L
- U4 pad 8: C3 -> GND L
- U4 pad 9: C4 -> unconnected-(U4-CHG_N-Pad9)
Routing:
- net +5V L: track 401.0 -> 0.00 mm, vias 28 -> 0
- net GND L: track 287.1 -> 0.00 mm, vias 45 -> 0
- net C3 L: track 258.0 -> 0.00 mm, vias 8 -> 0
- net C1 L: track 253.6 -> 0.00 mm, vias 8 -> 0
- net C2 L: track 226.2 -> 0.00 mm, vias 10 -> 0
- net C1: track 218.0 -> 0.00 mm, vias 16 -> 0
- net R2 L: track 214.9 -> 0.00 mm, vias 4 -> 0
- net +3.3V: track 206.9 -> 0.00 mm, vias 9 -> 0
- net C5: track 199.0 -> 0.00 mm, vias 11 -> 0
- net C4: track 195.9 -> 0.00 mm, vias 9 -> 0
- net R1: track 189.3 -> 0.00 mm
- net C2: track 188.5 -> 0.00 mm, vias 8 -> 0
- net C5 L: track 185.8 -> 0.00 mm, vias 13 -> 0
- net C4 L: track 182.7 -> 0.00 mm, vias 10 -> 0
- net +3.3V L: track 179.8 -> 0.00 mm, vias 6 -> 0
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- removed copper zone on B.Cu, net +5V
- removed copper zone on B.Cu, net +5V L
- removed copper zone on F.Cu, net GND
- removed copper zone on F.Cu, net GND L
Other:
- board size 281.7 x 89.1 mm -> 141 x 88.5 mm
- board text added: "9deg"
- board text removed: "Zboard V 0.4"
